File: blinkekatze-charger.kicad_pcb (KiCad board)
At the start: 4 copper layers, 397 parts, among them J1 USB_C_Receptacle, J10 USB_C_Receptacle, J11 USB_C_Receptacle, J12 USB_C_Receptacle, J13 USB_C_Receptacle, J14 USB_C_Receptacle, J15 USB_C_Receptacle, J16 USB_C_Receptacle, J17 USB_C_Receptacle_USB2.0, J18 USB_C_Receptacle, J19 USB_C_Receptacle, J2 USB_C_Receptacle, J20 USB_C_Receptacle, J21 USB_C_Receptacle, J3 USB_C_Receptacle, J4 USB_C_Receptacle, J5 USB_C_Receptacle, J6 USB_C_Receptacle, J7 USB_C_Receptacle, J8 USB_C_Receptacle, J9 USB_C_Receptacle, Q1 AON7534, Q2 AON7534, U1 MT9700, U10 MT9700, U11 AOZ1267QI, U12 MT9700, U13 MT9700, U14 MT9700, U15 MT9700, U16 AOZ1267QI, U17 MT9700, U18 MT9700, U19 MT9700, U2 AOZ1267QI, U20 MT9700, U21 CYPD3177, U22 AOZ1267QI, U23 MT9700, U24 MT9700, U25 MT9700, U26 MT9700, U3 MT9700, U4 MT9700, U5 MT9700, U6 AOZ1267QI, U7 MT9700, U8 MT9700, U9 MT9700

Commit message: Layout group 1 port 4
Parts:
- moved C26 199.4 mm to (167.9, 107.8), turned to -90 degrees
- moved R16 198.8 mm to (163.4, 107.2), turned to 180 degrees
- moved U5 197.1 mm to (160.4, 108.3), turned to -90 degrees
- moved F4 195.6 mm to (163.2, 110.2), turned to 90 degrees
- moved R18 192.8 mm to (169.4, 103.3), turned to 90 degrees
- moved R17 192.0 mm to (167.3, 101.1), turned to -90 degrees
- moved R19 191.1 mm to (170.4, 103.3), turned to 90 degrees
- moved C24 188.4 mm to (160.4, 111.5), turned to 180 degrees
- moved D4 182.9 mm to (169.2, 98.7), turned to -90 degrees
- moved FB7 180.8 mm to (165.1, 103.3), turned to 180 degrees
- moved C27 180.6 mm to (165.7, 100.1), turned to 90 degrees
- moved C25 179.5 mm to (160.4, 105.2), turned to 180 degrees
- moved FB8 176.9 mm to (160.0, 103.4), turned to 180 degrees
- moved C10 88.4 mm to (48.2, 108.6)
- moved C11 88.4 mm to (46.2, 108.6)
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Routing:
- net Net-(J2-CC2): track 4.85 -> 23.8 mm, vias 1 -> 2
- net Net-(U5-IN): track 0.00 -> 13.9 mm, vias 0 -> 2
- net Net-(J4-CC2): track 0.00 -> 13.6 mm, vias 0 -> 2
- net Net-(U3-IN): track 2.99 -> 16.1 mm, vias 1 -> 3
- net Net-(J4-CC1): track 0.00 -> 12.1 mm, vias 0 -> 2
- net Net-(J2-CC1): track 6.14 -> 18.2 mm, vias 1 -> 2
- net GND: track 18.7 -> 28.9 mm, vias 31 -> 52
- net Net-(U3-SET): track 0.95 -> 6.45 mm, vias 1 -> 2
- net Net-(U5-SET): track 0.00 -> 5.17 mm, vias 0 -> 2
- net Net-(D4-K): track 0.00 -> 3.81 mm, vias 0 -> 21
- net Net-(D4-A): track 0.00 -> 2.18 mm
- net Net-(C27-Pad1): track 0.00 -> 1.75 mm, vias 0 -> 9
- net Net-(C19-Pad1): vias 9 -> 16
- added copper zone on F.Cu, net Net-(C27-Pad1)
- added copper zone on In2.Cu, net Net-(C27-Pad1)
- added copper zone on F.Cu, net Net-(D4-K)
- added copper zone on In1.Cu, net Net-(D4-K)
- added copper zone on F.Cu, net Net-(U3-IN)
- added copper zone on F.Cu, net Net-(U3-OUT)
- added copper zone on F.Cu, net Net-(U5-IN)
- added copper zone on F.Cu, net Net-(U5-OUT)

Commit message: Finish group 1 layout
Parts:
- C122, C32, C59, C7, C86: value 100nF HV -> 100nF; footprint Capacitor_SMD:C_0603_1608Metric -> Capacitor_SMD:C_0402_1005Metric
- C123, C33, C5, C60, C87: value 100nF -> 1uF
- moved R12 178.6 mm to (153.1, 110.7), turned to 90 degrees
- moved C22 173.2 mm to (154.7, 106.1), turned to -90 degrees
- moved F3 173.2 mm to (150.0, 111.7)
- moved U4 171.8 mm to (149.5, 106.5), turned to -90 degrees
- moved R13 166.9 mm to (150.9, 101.1), turned to 90 degrees
- moved R15 164.2 mm to (152.5, 102.0), turned to 180 degrees
- moved R14 163.8 mm to (155.5, 98.8), turned to 90 degrees
- moved C20 163.0 mm to (149.5, 109.6), turned to 180 degrees
- moved C122 159.0 mm to (111.5, 44.9)
- moved D3 156.6 mm to (149.2, 98.7), turned to -90 degrees
- moved C32 154.2 mm to (111.5, 37.0)
- moved C21 154.0 mm to (149.5, 103.4), turned to 180 degrees
- moved C23 153.9 mm to (145.7, 100.1), turned to 90 degrees
- moved FB5 153.8 mm to (153.2, 100.2), turned to 180 degrees
- moved FB6 149.4 mm to (153.2, 98.5)
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Routing:
- net GND: track 28.9 -> 54.0 mm, vias 52 -> 93
- net Net-(J3-CC1): track 0.00 -> 19.3 mm, vias 0 -> 2
- net Net-(U4-IN): track 0.00 -> 14.6 mm, vias 0 -> 4
- net Net-(J3-CC2): track 0.00 -> 13.8 mm, vias 0 -> 2
- net Net-(U4-SET): track 0.00 -> 8.13 mm, vias 0 -> 2
- net /Port group 1/VCC: track 0.00 -> 7.05 mm, vias 0 -> 2
- net /Port group 1/Port 1/VIN: track 0.00 -> 5.00 mm, vias 0 -> 26
- net Net-(U2-FB): track 0.00 -> 4.31 mm
- net IN: track 0.00 -> 2.09 mm
- net Net-(D3-A): track 0.00 -> 1.89 mm
- net Net-(U2-BST): track 0.00 -> 1.73 mm
- net Net-(C7-Pad2): track 0.00 -> 1.67 mm
- net Net-(U2-SS): track 0.00 -> 1.66 mm
- net Net-(U2-TON): track 0.00 -> 1.55 mm
- net Net-(C23-Pad1): track 0.00 -> 1.33 mm, vias 0 -> 12
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- added copper zone on B.Cu, net /Port group 1/Port 1/VIN
- added copper zone on F.Cu, net /Port group 1/Port 1/VIN
- added copper zone on F.Cu, net /Port group 1/VIN
- added copper zone on In2.Cu, net /Port group 1/VIN
- added copper zone on In1.Cu, net GND
- added copper zone on F.Cu, net IN
- added copper zone on F.Cu, net Net-(C23-Pad1)
- added copper zone on In2.Cu, net Net-(C23-Pad1)
- added copper zone on F.Cu, net Net-(C7-Pad2)
- added copper zone on F.Cu, net Net-(D3-K)
- added copper zone on In1.Cu, net Net-(D3-K)
- added copper zone on F.Cu, net Net-(U4-IN)
- added copper zone on F.Cu, net Net-(U4-OUT)
