File: blinkekatze-charger.kicad_sch (KiCad schematic)
At the start: 27 parts, among them J2 USB_C_Receptacle_USB2.0, Q1 AON7534, U2 CYPD3177

Commit message: Finish layout
Parts:
- removed C9: 1nF, Capacitor_SMD:C_1206_3216Metric, symbol Device:C_Small
- removed R3: 100k HV, Resistor_SMD:R_1206_3216Metric, symbol Device:R_Small
- added H1: M3, MountingHole:MountingHole_3.2mm_M3, symbol Mechanical:MountingHole
- added H2, H3: ToolingHole, ToolingHole:ToolingHole_JLCSMT, symbol Mechanical:MountingHole
Connections:
- net GND: now also J2.S1 (SHIELD)

Commit message: Consolidate bom items
Parts:
- H1, H2, H3: now left out of the parts list
- R4: value 100k -> 1M; LCSC C25741 -> C26083
- R4: value 10k -> 100k; LCSC C25744 -> C25741

Commit message: Advertise all charging ports as DCP
Parts:
- Q1: value AON7534 -> AP90P03Q; LCSC C115844 -> C2849567
